Commit message: ;

File: indy7_robotiq_description/urdf/indy7_robotiq.xacro (robot description, xacro)
@@ -1,8 +1,6 @@
 <?xml version="1.0" ?>
 <robot name="indy7_and_robotiq" xmlns:xacro="http://ros.org/wiki/xacro">
+  <xacro:include filename="$(find indy7_description)/urdf/indy7.xacro"/>
   <xacro:include filename="$(find indy7_robotiq_description)/urdf/robotiq_arg85_description.xacro"/>
-  <xacro:include filename="$(find indy7_description)/urdf/indy7.xacro"/>
-  <!-- <xacro:indy7/> -->
-  <xacro:robotiq_arg85 connected_to="tcp"/>
   <joint name="indy7_joint_tcp" type="fixed">
     <parent link="tcp"/>

File: indy7_robotiq_description/urdf/robotiq_arg85_description.xacro (robot description, xacro)
@@ -1,5 +1,4 @@
 <?xml version="1.0" ?>
 <robot xmlns:xacro="http://www.ros.org/wiki/xacro" name="robotiq_arg85_description">
-<xacro:macro name="robotiq_arg85" params="arm_id:='indy7' connected_to:='' xyz:='0 0 0' rpy:='0 0 0'">
   <link name="robotiq_85_base_link">
     <inertial>
@@ -497,4 +496,3 @@
       xyz="0 1 0" />
   </joint>
-</xacro:macro>
 </robot>
